Commit message: Add solid Tesollo palm collision core

File: assets/robot_hands/direct_motor/tesollo_dg5f/left/hand.urdf (robot description, URDF)
Before this commit: robot tesollo_dg5f_left_direct_motor, 28 links, 27 joints
Links:
- link ll_dg_palm: geometry collision box size=0.045 0.055 0.07; collision mesh filename=meshes/0005_ll_dg_palm_c_00.obj

File: assets/robot_hands/direct_motor/tesollo_dg5f/right/hand.urdf (robot description, URDF)
Before this commit: robot tesollo_dg5f_right_direct_motor, 28 links, 27 joints
Links:
- link rl_dg_palm: geometry collision box size=0.045 0.055 0.07; collision mesh filename=meshes/0005_rl_dg_palm_c_00.obj

Commit message: Fill Tesollo base to palm visual gap

File: assets/robot_hands/direct_motor/tesollo_dg5f/left/hand.urdf (robot description, URDF)
Before this commit: robot tesollo_dg5f_left_direct_motor, 28 links, 27 joints
Links:
- link ll_dg_base: geometry collision box size=0.045 0.055 0.087; collision mesh filename=meshes/0003_ll_dg_base_c_00.obj

File: assets/robot_hands/direct_motor/tesollo_dg5f/right/hand.urdf (robot description, URDF)
Before this commit: robot tesollo_dg5f_right_direct_motor, 28 links, 27 joints
Links:
- link rl_dg_base: geometry collision box size=0.045 0.055 0.087; collision mesh filename=meshes/0003_rl_dg_base_c_00.obj
